File: hardware/Drone_board/Drone_board.kicad_sch (KiCad schematic)
At the start: 12 parts, among them J1 Conn_01x08_Pin, J2 Conn_01x03_Pin, J3 Conn_01x03_Pin, J4 Conn_01x03_Pin, J5 Conn_01x03_Pin, J6 Conn_01x03_Pin, J7 Conn_01x03_Pin, U1 NUCLEO-L432KC, U3 NRF24L01_Breakout

Commit message: Schematic drone for validation
Parts:
- removed J3: Conn_01x03_Pin, symbol Connector:Conn_01x03_Pin
- added D1: Red_LED, symbol Device:LED
- added D2: Green_LED, symbol Device:LED
- added J3: Conn_01x04_Pin, symbol Connector:Conn_01x04_Pin
- added Q1: 2N2219, Package_TO_SOT_THT:TO-39-3, symbol Transistor_BJT:2N2219
- added R1: 455, symbol Device:R
- added R2: 405, symbol Device:R
- added R3: 2000, symbol Device:R
- added R4: 510, symbol Device:R
Connections:
- net GND: now also D1.1 (K), D2.1 (K), J3.1 (Pin_1), J3.4 (Pin_4), Q1.3 (C), R1.2, R2.2, R4.2
- net GPIO_EXT_MPU: now also U1.CN3_14 (PB5); no longer U1.CN3_2 (PA10)
- net MOSI_NRF: now also U1.CN3_5 (PA12); no longer U1.CN4_6 (PA7)
- net TIM_PWM1: now reaches J4.2 (Pin_2)
- net TIM_PWM1: now also U1.CN3_12 (PA8)
- net PWM_Neopixel: now reaches U1.CN4_12 (PA0)
- net PWM_Neopixel: now also J2.2 (Pin_2)
- net Battery_ADC: now reaches U1.CN4_8 (PA5)
- net Battery_ADC: now also R3.2, R4.1
- net Battery_set: now reaches U1.CN4_9 (PA4)
- net Battery_set: now also Q1.2 (B)
- net TIM_PWM4: now reaches J7.2 (Pin_2)
- net TIM_PWM4: now also U1.CN3_13 (PA11)
- net TIM_PWM3: now reaches J6.2 (Pin_2)
- net TIM_PWM3: now also U1.CN3_2 (PA10)
- net GPIO_EXT_NRF: now reaches U3.8 (IRQ)
- net GPIO_EXT_NRF: now also U1.CN3_8 (PB6)
- net I2C_SDA_MPU: now reaches U1.CN3_15 (PB4)
- net I2C_SDA_MPU: now also J1.4 (Pin_4)
- net TIM_PWM2: now reaches J5.2 (Pin_2)
- net TIM_PWM2: now also U1.CN3_1 (PA9)
- net SCL_MPU renamed I2C_SCL_MPU
- net I2C_SCL_MPU: now also U1.CN4_6 (PA7); no longer U1.CN3_1 (PA9)
- net SDA_MPU: no longer names the net of U1.CN3_7 (PB7)
- net SDA_MPU: no longer J1.4 (Pin_4)
- new net: Q1.1 (E), R3.1
- new net: D2.2 (A), R2.1
- new net: D1.2 (A), R1.1
- no-connect marks 6 -> 14
Other:
- moved on the sheet: C1, C2, C3, J1, J2, J4, J5, J6, J7, U1A, U1B, U3

Commit message: Board schematic validate
Parts:
- removed C1: 100u, symbol Device:C_Small
- removed C2, C3: 100u, symbol Device:C
- removed D1: Red_LED, symbol Device:LED
- removed D2: Green_LED, symbol Device:LED
- removed Q1: 2N2219, Package_TO_SOT_THT:TO-39-3, symbol Transistor_BJT:2N2219
- added C4: 1OOu, symbol Device:C_Polarized_Small
- added C5: 100u, symbol Device:C_Polarized_Small
- added D1: LED_RED, symbol Device:LED_Small
- added D2: LED_GREEN, symbol Device:LED_Small
- added H1, H2, H5, H6: MountingHole_Pad, MountingHole:MountingHole_3.2mm_M3_Pad_Via, symbol Mechanical:MountingHole_Pad
- J1: footprint (none) -> Connector_PinHeader_2.54mm:PinHeader_1x08_P2.54mm_Vertical
- J2, J4, J5, J6, J7: footprint (none) -> Connector_PinHeader_2.54mm:PinHeader_1x03_P2.54mm_Vertical
- J3: footprint (none) -> Connector_JST:JST_XH_B4B-XH-A_1x04_P2.50mm_Vertical
- R1: value 455 -> 1000
- R2: value 405 -> 1000
- R3: value 2000 -> 200000
- R4: value 510 -> 51000
Connections:
- net 3,3V is gone; now on net VCC_3V3: U1.CN4_14 (+3V3)
- net Battery_set is gone; now on an unnamed net: U1.CN4_9 (PA4)
- net GND: now also C4.2, C5.2, D1.1 (K), D2.1 (K), H1.1, H2.1, H5.1, H6.1; no longer J3.1 (Pin_1), R1.2, R2.2
- net VCC_5_MPU: now also J1.1 (Pin_1), C4.1
- net VCC_5_NEO: now also J2.3 (Pin_3)
- net at R3.1: now also J3.1 (Pin_1)
- net at U1.CN4_10 (PA3): now also R1.1
- net VCC_3V3: now reaches U3.2 (VCC)
- net VCC_3V3: now also C5.1
- net +5V renamed VCC_5V_STM
- new net: D1.2 (A), R1.2
- new net: D2.2 (A), R2.2
- no-connect marks 14 -> 15
Other:
- moved on the sheet: J1, J2, J3, J4, J5, J6, J7, R3, R4, U3

Commit message: PCB Footprint
Parts:
- C4, C5: footprint (none) -> Capacitor_SMD:C_0805_2012Metric
- D1, D2: footprint (none) -> LED_SMD:LED_0603_1608Metric_Pad1.05x0.95mm_HandSolder
- R1, R2, R3, R4: footprint (none) -> Resistor_SMD:R_0805_2012Metric_Pad1.20x1.40mm_HandSolder
Changed lines of the file:
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@@
       (effects (font (size 1.27 1.27)) (justify left))
     )
-    (property "Footprint" "" (at 189.992 55.88 90)
+    (property "Footprint" "Resistor_SMD:R_0805_2012Metric_Pad1.20x1.40mm_HandSolder" (at 189.992 55.88 90)
       (effects (font (size 1.27 1.27)) hide)
     )
@@
       (effects (font (size 1.27 1.27)))
     )
-    (property "Footprint" "" (at 40.64 60.452 90)
+    (property "Footprint" "Resistor_SMD:R_0805_2012Metric_Pad1.20x1.40mm_HandSolder" (at 40.64 60.452 90)
       (effects (font (size 1.27 1.27)) hide)
     )
@@
       (effects (font (size 1.27 1.27)) (justify left))
     )
-    (property "Footprint" "" (at 189.992 44.45 90)
+    (property "Footprint" "Resistor_SMD:R_0805_2012Metric_Pad1.20x1.40mm_HandSolder" (at 189.992 44.45 90)
       (effects (font (size 1.27 1.27)) hide)
     )
@@
       (effects (font (size 1.27 1.27)) (justify left))
     )
-    (property "Footprint" "" (at 154.94 36.83 0)
+    (property "Footprint" "Capacitor_SMD:C_0805_2012Metric" (at 154.94 36.83 0)
       (effects (font (size 1.27 1.27)) hide)
     )
@@
       (effects (font (size 1.27 1.27)) (justify right))
     )
-    (property "Footprint" "" (at 34.29 66.04 90)
+    (property "Footprint" "LED_SMD:LED_0603_1608Metric_Pad1.05x0.95mm_HandSolder" (at 34.29 66.04 90)
       (effects (font (size 1.27 1.27)) hide)
     )
@@
       (effects (font (size 1.27 1.27)))
     )
-    (property "Footprint" "" (at 95.25 56.388 90)
+    (property "Footprint" "Resistor_SMD:R_0805_2012Metric_Pad1.20x1.40mm_HandSolder" (at 95.25 56.388 90)
       (effects (font (size 1.27 1.27)) hide)
     )
@@
       (effects (font (size 1 1)) (justify left))
     )
-    (property "Footprint" "" (at 170.18 99.06 0)
+    (property "Footprint" "Capacitor_SMD:C_0805_2012Metric" (at 170.18 99.06 0)
       (effects (font (size 1.27 1.27)) hide)
     )
@@
       (effects (font (size 1.27 1.27)) (justify right))
     )
-    (property "Footprint" "" (at 99.06 63.5 90)
-      (effects (font (size 1.27 1.27)) hide)
-    )
+    (property "Footprint" "LED_SMD:LED_0603_1608Metric_Pad1.05x0.95mm_HandSolder" (at 99.06 63.5 90)
+      (effects (font (size 1.27 1.27)) hide)
+    )

Commit message: PCB footprint
Parts:
- C4, C5: footprint Capacitor_SMD:C_0805_2012Metric -> Capacitor_SMD:CP_Elec_6.3x7.7
- H1, H2, H5, H6: footprint MountingHole:MountingHole_3.2mm_M3_Pad_Via -> MountingHole:MountingHole_3.2mm_M3_Pad
- R1, R2, R3, R4: footprint Resistor_SMD:R_0805_2012Metric_Pad1.20x1.40mm_HandSolder -> Resistor_SMD:R_0603_1608Metric
Changed lines of the file:
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@@
     (stroke (width 0) (type default))
   )
-  (wire (pts (xy 82.55 36.83) (xy 78.74 36.83))
+  (wire (pts (xy 83.82 36.83) (xy 78.74 36.83))
     (stroke (width 0) (type default))
   )
@@
     (effects (font (size 1.27 1.27)) (justify left bottom))
   )
-  (label "VCC_5V_STM" (at 82.55 36.83 0) (fields_autoplaced)
+  (label "VCC_5V_STM" (at 83.82 36.83 0) (fields_autoplaced)
     (effects (font (size 1.27 1.27)) (justify left bottom))
   )
@@
       (effects (font (size 1.27 1.27)) (justify left))
     )
-    (property "Footprint" "Resistor_SMD:R_0805_2012Metric_Pad1.20x1.40mm_HandSolder" (at 189.992 55.88 90)
+    (property "Footprint" "Resistor_SMD:R_0603_1608Metric" (at 189.992 55.88 90)
       (effects (font (size 1.27 1.27)) hide)
     )
@@
       (effects (font (size 1.27 1.27)))
     )
-    (property "Footprint" "Resistor_SMD:R_0805_2012Metric_Pad1.20x1.40mm_HandSolder" (at 40.64 60.452 90)
+    (property "Footprint" "Resistor_SMD:R_0603_1608Metric" (at 40.64 60.452 90)
       (effects (font (size 1.27 1.27)) hide)
     )
@@
       (effects (font (size 1.27 1.27)) (justify left))
     )
-    (property "Footprint" "Resistor_SMD:R_0805_2012Metric_Pad1.20x1.40mm_HandSolder" (at 189.992 44.45 90)
+    (property "Footprint" "Resistor_SMD:R_0603_1608Metric" (at 189.992 44.45 90)
       (effects (font (size 1.27 1.27)) hide)
     )
@@
       (effects (font (size 1.27 1.27)) (justify left))
     )
-    (property "Footprint" "MountingHole:MountingHole_3.2mm_M3_Pad_Via" (at 128.27 146.05 0)
+    (property "Footprint" "MountingHole:MountingHole_3.2mm_M3_Pad" (at 128.27 146.05 0)
       (effects (font (size 1.27 1.27)) hide)
     )
@@
       (effects (font (size 1.27 1.27)) (justify left))
     )
-    (property "Footprint" "Capacitor_SMD:C_0805_2012Metric" (at 154.94 36.83 0)
+    (property "Footprint" "Capacitor_SMD:CP_Elec_6.3x7.7" (at 154.94 36.83 0)
       (effects (font (size 1.27 1.27)) hide)
     )
@@
     )
   )
+  (symbol (lib_id "Connector:Conn_01x03_Pin") (at 31.75 143.51 0) (unit 1)
+    (in_bom yes) (on_board yes) (dnp no)
+    (property "Reference" "J4" (at 32.385 137.16 0)
+      (effects (font (size 1.27 1.27)))
+    )
+    (property "Value" "Conn_01x03_Pin" (at 36.83 158.75 0)
+      (effects (font (size 1.27 1.27)))
+    )
+    (property "Footprint" "Connector_PinHeader_2.54mm:PinHeader_1x03_P2.54mm_Vertical" (at 31.75 143.51 0)
+      (effects (font (size 1.27 1.27)) hide)
+    )
+    (property "Datasheet" "~" (at 31.75 143.51 0)
+      (effects (font (size 1.27 1.27)) hide)
+    )
+    (pin "1")
+    (pin "2")
+    (pin "3")
+    (instances
+      (project "Drone_board"
+        (path "/73528b15-87bf-4854-86cb-863685c61d6c"
+          (reference "J4") (unit 1)
+        )
+      )
+    )
+  )
   (symbol (lib_id "power:GND") (at 140.97 72.39 0) (unit 1)
     (in_bom yes) (on_board yes) (dnp no) (fields_autoplaced)
@@
         (path "/73528b15-87bf-4854-86cb-863685c61d6c"
           (reference "#PWR03") (unit 1)
-        )
-      )
-    )
-  )
-  (symbol (lib_id "Connector:Conn_01x03_Pin") (at 31.75 143.51 0) (unit 1)
-    (in_bom yes) (on_board no) (dnp no)
-    (property "Reference" "J4" (at 32.385 137.16 0)
-      (effects (font (size 1.27 1.27)))
-    )
-    (property "Value" "Conn_01x03_Pin" (at 36.83 158.75 0)
-      (effects (font (size 1.27 1.27)))
-    )
-    (property "Footprint" "Connector_PinHeader_2.54mm:PinHeader_1x03_P2.54mm_Vertical" (at 31.75 143.51 0)
-      (effects (font (size 1.27 1.27)) hide)
-    )
-    (property "Datasheet" "~" (at 31.75 143.51 0)
-      (effects (font (size 1.27 1.27)) hide)
-    )
-    (pin "1")
-    (pin "2")
-    (pin "3")
-    (instances
-      (project "Drone_board"
-        (path "/73528b15-87bf-4854-86cb-863685c61d6c"
-          (reference "J4") (unit 1)
         )
       )
@@
       (effects (font (size 1.27 1.27)) (justify left))
     )
-    (property "Footprint" "MountingHole:MountingHole_3.2mm_M3_Pad_Via" (at 128.27 138.43 0)
+    (property "Footprint" "MountingHole:MountingHole_3.2mm_M3_Pad" (at 128.27 138.43 0)
       (effects (font (size 1.27 1.27)) hide)
     )
@@
       (effects (font (size 1.27 1.27)) (justify left))
     )
-    (property "Footprint" "MountingHole:MountingHole_3.2mm_M3_Pad_Via" (at 128.27 153.67 0)
+    (property "Footprint" "MountingHole:MountingHole_3.2mm_M3_Pad" (at 128.27 153.67 0)
       (effects (font (size 1.27 1.27)) hide)
     )
@@
       (effects (font (size 1.27 1.27)))
     )
-    (property "Footprint" "Resistor_SMD:R_0805_2012Metric_Pad1.20x1.40mm_HandSolder" (at 95.25 56.388 90)
+    (property "Footprint" "Resistor_SMD:R_0603_1608Metric" (at 95.25 56.388 90)
       (effects (font (size 1.27 1.27)) hide)
     )
@@
       (effects (font (size 1 1)) (justify left))
     )
-    (property "Footprint" "Capacitor_SMD:C_0805_2012Metric" (at 170.18 99.06 0)
+    (property "Footprint" "Capacitor_SMD:CP_Elec_6.3x7.7" (at 170.18 99.06 0)
       (effects (font (size 1.27 1.27)) hide)
     )
@@
       (effects (font (size 1.27 1.27)) (justify left))
     )
-    (property "Footprint" "MountingHole:MountingHole_3.2mm_M3_Pad_Via" (at 128.27 160.02 0)
-      (effects (font (size 1.27 1.27)) hide)
-    )
+    (property "Footprint" "MountingHole:MountingHole_3.2mm_M3_Pad" (at 128.27 160.02 0)
+      (effects (font (size 1.27 1.27)) hide)
+    )
