File: hardware/Drone_board/Drone_board.kicad_pcb (KiCad board)
At the start: 2 copper layers, 1 part, among them U1 NUCLEO-L432KC

Commit message: Board schematic validate
Parts:
- added H1: MountingHole_Pad, MountingHole:MountingHole_3.2mm_M3_Pad_Via, F.Cu at (33.5, 50.9)
- added H2: MountingHole_Pad, MountingHole:MountingHole_3.2mm_M3_Pad_Via, F.Cu at (33.5, 58.8)
- added H5: MountingHole_Pad, MountingHole:MountingHole_3.2mm_M3_Pad_Via, F.Cu at (33.5, 66.8)
- added H6: MountingHole_Pad, MountingHole:MountingHole_3.2mm_M3_Pad_Via, F.Cu at (33.5, 74.7)
- added J1: Conn_01x08_Pin, Connector_PinHeader_2.54mm:PinHeader_1x08_P2.54mm_Vertical, F.Cu at (39.8, 58.9)
- added J2: Conn_01x03_Pin, Connector_PinHeader_2.54mm:PinHeader_1x03_P2.54mm_Vertical, F.Cu at (39.8, 49.2)
- added J3: Conn_01x04_Pin, Connector_JST:JST_XH_B4B-XH-A_1x04_P2.50mm_Vertical, F.Cu at (45.6, 60.0)
- added J5: Conn_01x03_Pin, Connector_PinHeader_2.54mm:PinHeader_1x03_P2.54mm_Vertical, F.Cu at (44.5, 49.2)
- added J6: Conn_01x03_Pin, Connector_PinHeader_2.54mm:PinHeader_1x03_P2.54mm_Vertical, F.Cu at (49.1, 49.2)
- added J7: Conn_01x03_Pin, Connector_PinHeader_2.54mm:PinHeader_1x03_P2.54mm_Vertical, F.Cu at (53.8, 49.2)
- added Q1: 2N2219, Package_TO_SOT_THT:TO-39-3, F.Cu at (73.9, 82.5)
- added U3: NRF24L01_Breakout, RF_Module:nRF24L01_Breakout, F.Cu at (80.0, 35.1)
- moved U1 15.8 mm to (120.5, 89.9)
Connections:
- U1 pad CN3_1: unconnected-(U1A-PA9-PadCN3_1) -> /TIM_PWM2
- U1 pad CN3_12: unconnected-(U1A-PA8-PadCN3_12) -> /TIM_PWM1
- U1 pad CN3_13: unconnected-(U1A-PA11-PadCN3_13) -> /TIM_PWM4
- U1 pad CN3_14: unconnected-(U1A-PB5-PadCN3_14) -> /GPIO_EXT_MPU
- U1 pad CN3_15: unconnected-(U1A-PB4-PadCN3_15) -> /I2C_SDA_MPU
- U1 pad CN3_2: unconnected-(U1A-PA10-PadCN3_2) -> /TIM_PWM3
- U1 pad CN3_4: unconnected-(U1A-GND_CN3-PadCN3_4) -> GND
- U1 pad CN3_5: unconnected-(U1A-PA12-PadCN3_5) -> /MOSI_NRF
- U1 pad CN3_6: unconnected-(U1A-PB0-PadCN3_6) -> /CSN_NRF
- U1 pad CN3_8: unconnected-(U1A-PB6-PadCN3_8) -> /GPIO_EXT_NRF
- U1 pad CN3_9: unconnected-(U1A-PB1-PadCN3_9) -> /CE_NRF
- U1 pad CN4_1: (no net) -> unconnected-(U1B-VIN-PadCN4_1)
- U1 pad CN4_10: (no net) -> Net-(U1B-PA3)
- U1 pad CN4_11: (no net) -> /SCK_NRF
- U1 pad CN4_12: (no net) -> /PWM_Neopixel
- U1 pad CN4_13: (no net) -> unconnected-(U1B-AREF-PadCN4_13)
- U1 pad CN4_14: (no net) -> /VCC_3V3
- U1 pad CN4_15: (no net) -> unconnected-(U1B-PB3-PadCN4_15)
- U1 pad CN4_2: (no net) -> GND
- U1 pad CN4_3: (no net) -> unconnected-(U1B-NRST_CN4-PadCN4_3)
- U1 pad CN4_4: (no net) -> /VCC_5V_STM
- U1 pad CN4_5: (no net) -> unconnected-(U1B-PA2-PadCN4_5)
- U1 pad CN4_6: (no net) -> /I2C_SCL_MPU
- U1 pad CN4_7: (no net) -> /MISO_NRF
- U1 pad CN4_8: (no net) -> Battery_ADC
- U1 pad CN4_9: (no net) -> Net-(U1B-PA4)
Routing:
- added copper zone on F.Cu, net GND

Commit message: PCB Footprint
Parts:
- removed Q1: 2N2219, Package_TO_SOT_THT:TO-39-3
- added C4: 1OOu, Capacitor_SMD:C_0805_2012Metric, F.Cu at (207.7, 83.0)
- added C5: 100u, Capacitor_SMD:C_0805_2012Metric, F.Cu at (207.7, 86.0)
- added D1: LED_RED, LED_SMD:LED_0603_1608Metric_Pad1.05x0.95mm_HandSolder, F.Cu at (195.0, 88.5)
- added D2: LED_GREEN, LED_SMD:LED_0603_1608Metric_Pad1.05x0.95mm_HandSolder, F.Cu at (195.0, 91.1)
- added R1: 1000, Resistor_SMD:R_0805_2012Metric_Pad1.20x1.40mm_HandSolder, F.Cu at (195.2, 76.9)
- added R2: 1000, Resistor_SMD:R_0805_2012Metric_Pad1.20x1.40mm_HandSolder, F.Cu at (195.2, 79.8)
- added R3: 200000, Resistor_SMD:R_0805_2012Metric_Pad1.20x1.40mm_HandSolder, F.Cu at (195.2, 82.8)
- added R4: 51000, Resistor_SMD:R_0805_2012Metric_Pad1.20x1.40mm_HandSolder, F.Cu at (195.2, 85.7)
- moved J1 151.1 mm to (190.5, 69.9)
- moved J2 151.1 mm to (190.5, 60.2)
- moved J5 151.1 mm to (195.1, 60.2)
- moved J3 151.1 mm to (196.3, 71.0)
- moved J6 151.1 mm to (199.8, 60.2)
- moved J7 151.1 mm to (204.4, 60.2)
- moved U3 102.9 mm to (182.5, 43.9)
- moved H5 100.6 mm to (130.4, 39.8)
- moved H6 100.5 mm to (131.2, 98.2)
- moved U1 54.7 mm to (170.2, 67.0)
- moved H2 40.4 mm to (42.3, 98.2)
- moved H1 15.3 mm to (44.0, 39.8)
Routing:
- removed copper zone on F.Cu, net GND

Commit message: PCB footprint
Parts:
- added J4: Conn_01x03_Pin, Connector_PinHeader_2.54mm:PinHeader_1x03_P2.54mm_Vertical, F.Cu at (79.0, 62.5)
- C4, C5: footprint Capacitor_SMD:C_0805_2012Metric -> Capacitor_SMD:CP_Elec_6.3x7.7
- H1, H2, H5, H6: footprint MountingHole:MountingHole_3.2mm_M3_Pad_Via -> MountingHole:MountingHole_3.2mm_M3_Pad
- R1, R2: footprint Resistor_SMD:R_0805_2012Metric_Pad1.20x1.40mm_HandSolder -> Resistor_SMD:R_0603_1608Metric
- R3, R4: footprint Resistor_SMD:R_0805_2012Metric_Pad1.20x1.40mm_HandSolder -> Resistor_SMD:R_0603_1608Metric; moved to B.Cu
- U1: moved to B.Cu
- moved J6 134.2 mm to (66.0, 70.0)
- moved J2 124.6 mm to (66.0, 55.0)
- moved C5 122.4 mm to (90.8, 49.5)
- moved R1 115.4 mm to (80.0, 84.0)
- moved R2 115.4 mm to (80.0, 86.5)
- moved D1 115.1 mm to (80.0, 91.0)
- moved D2 115.1 mm to (80.0, 93.6)
- moved C4 111.5 mm to (101.3, 49.5), turned to 180 degrees
- moved R3 109.7 mm to (87.0, 101.0), turned to 180 degrees
- moved R4 109.6 mm to (87.0, 103.5), turned to 180 degrees
- moved J3 109.4 mm to (92.0, 104.0)
- moved J1 95.5 mm to (95.0, 67.0)
- moved J7 93.8 mm to (113.5, 83.0)
- moved U3 92.1 mm to (90.4, 43.0), turned to 90 degrees
- moved H2 88.7 mm to (111.0, 42.0)
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Routing:
- net /VCC_3V3: track 0.00 -> 57.7 mm
- net /VCC_5V_STM: track 0.00 -> 9.22 mm
- net /VCC_5_MPU: track 0.00 -> 9.00 mm
- added copper zone on F.Cu, net (none)
- added copper zone on B.Cu, net GND
Other:
- board outline added: 38 x 68 mm
- rule pad_to_mask_clearance: 0 -> 0.1

Commit message: Update PCB
Parts:
- moved J6 48.2 mm to (113.5, 62.0)
- moved J2 13.2 mm to (79.0, 57.0)
- moved J4 9.00 mm to (79.0, 71.5)
- moved D1 4.12 mm to (79.0, 95.0), turned to 90 degrees
- moved R1 3.95 mm to (79.0, 87.8), turned to -90 degrees
- moved C5 3.80 mm to (87.0, 49.5)
- moved R3 2.38 mm to (87.5, 103.3), turned to 90 degrees
- moved D2 2.13 mm to (81.6, 95.0), turned to 90 degrees
- moved J1 2.00 mm to (95.0, 65.0)
- moved R2 1.90 mm to (81.5, 87.7), turned to -90 degrees
- moved R4 1.51 mm to (85.5, 103.3), turned to -90 degrees
- moved C4 0.10 mm to (101.2, 49.5)
Routing:
- net /TIM_PWM1: track 0.00 -> 59.4 mm, vias 0 -> 2
- net /VCC_5_NEO: track 0.00 -> 51.6 mm, vias 0 -> 6
- net /CSN_NRF: track 0.00 -> 42.5 mm
- net /MOSI_NRF: track 0.00 -> 42.3 mm, vias 0 -> 2
- net /SCK_NRF: track 0.00 -> 41.4 mm, vias 0 -> 1
- net /GPIO_EXT_NRF: track 0.00 -> 40.8 mm, vias 0 -> 1
- net /CE_NRF: track 0.00 -> 37.4 mm
- net Battery_ADC: track 0.00 -> 34.0 mm, vias 0 -> 1
- net /MISO_NRF: track 0.00 -> 33.0 mm, vias 0 -> 2
- net /PWM_Neopixel: track 0.00 -> 28.3 mm
- net GND: track 0.00 -> 25.1 mm
- net /I2C_SDA_MPU: track 0.00 -> 24.2 mm
- net /VCC_5_MPU: track 9.00 -> 29.8 mm
- net Net-(U1B-PA3): track 0.00 -> 16.8 mm, vias 0 -> 2
- net Net-(U1B-PA4): track 0.00 -> 16.8 mm
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
Commit message: PCB validated by refrent
Routing:
- net GND: vias 0 -> 9
- net Battery_ADC: vias 1 -> 0
- added copper zone on F.Cu, net GND
- removed copper zone on F.Cu, net (none)
Changed lines of the file:
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@@
   (gr_arc (start 111 38) (mid 113.828427 39.171573) (end 115 42)
     (stroke (width 0.1) (type default)) (layer "Edge.Cuts"))
-  (dimension (type aligned) (layer "Edge.Cuts")
+  (dimension (type aligned) (layer "User.2")
     (pts (xy 81 42) (xy 81 102))
     (height 21)
-    (gr_text "60.0000 mm" (at 58.85 72 90) (layer "Edge.Cuts")
+    (gr_text "60.0000 mm" (at 58.85 72 90) (layer "User.2")
       (effects (font (size 1 1) (thickness 0.15)))
     )
@@
     (style (thickness 0.1) (arrow_length 1.27) (text_position_mode 0) (extension_height 0.58642) (extension_offset 0.5) keep_text_aligned)
   )
-  (dimension (type aligned) (layer "Edge.Cuts")
+  (dimension (type aligned) (layer "User.2")
     (pts (xy 81 102) (xy 111 102))
     (height 23)
-    (gr_text "30.0000 mm" (at 96 123.85) (layer "Edge.Cuts")
+    (gr_text "30.0000 mm" (at 96 123.85) (layer "User.2")
       (effects (font (size 1 1) (thickness 0.15)))
     )
@@
   (segment (start 81.59 95.875) (end 79 95.875) (width 0.5) (layer "F.Cu") (net 1))
   (segment (start 79 100) (end 79 95.875) (width 0.5) (layer "F.Cu") (net 1))
+  (via (at 94.9 91) (size 0.8) (drill 0.4) (layers "F.Cu" "B.Cu") (free) (net 1))
+  (via (at 96.6 98.3) (size 0.8) (drill 0.4) (layers "F.Cu" "B.Cu") (free) (net 1))
+  (via (at 100.3 67.8) (size 0.8) (drill 0.4) (layers "F.Cu" "B.Cu") (free) (net 1))
+  (via (at 82.5 69.6) (size 0.8) (drill 0.4) (layers "F.Cu" "B.Cu") (free) (net 1))
+  (via (at 80.8 51.5) (size 0.8) (drill 0.4) (layers "F.Cu" "B.Cu") (free) (net 1))
+  (via (at 85 57) (size 0.8) (drill 0.4) (layers "F.Cu" "B.Cu") (free) (net 1))
+  (via (at 101 81.4) (size 0.8) (drill 0.4) (layers "F.Cu" "B.Cu") (free) (net 1))
+  (via (at 108.2 75.4) (size 0.8) (drill 0.4) (layers "F.Cu" "B.Cu") (free) (net 1))
+  (via (at 100.4 42) (size 0.8) (drill 0.4) (layers "F.Cu" "B.Cu") (free) (net 1))
   (segment (start 111 52.04) (end 113 52.04) (width 0.75) (layer "F.Cu") (net 2))
   (segment (start 103.24 55) (end 108.04 55) (width 0.75) (layer "F.Cu") (net 2))
@@
   (segment (start 99 74.5) (end 99 89) (width 0.5) (layer "F.Cu") (net 15))
   (segment (start 95 72.62) (end 97.12 72.62) (width 0.5) (layer "F.Cu") (net 15))
+  (segment (start 83.38 62.62) (end 88 62.62) (width 0.5) (layer "F.Cu") (net 18))
   (segment (start 79 71) (end 79 67) (width 0.5) (layer "F.Cu") (net 18))
-  (segment (start 87.88 62.5) (end 88 62.62) (width 1) (layer "F.Cu") (net 18))
   (segment (start 79 67) (end 83.38 62.62) (width 0.5) (layer "F.Cu") (net 18))
-  (segment (start 83.38 62.62) (end 88 62.62) (width 0.5) (layer "F.Cu") (net 18))
-  (segment (start 87.88 62.5) (end 88 62.62) (width 1) (layer "B.Cu") (net 18))
   (segment (start 88 67.7) (end 91.2 67.7) (width 0.5) (layer "B.Cu") (net 20))
   (segment (start 93.58 70.08) (end 95 70.08) (width 0.5) (layer "B.Cu") (net 20))
@@
   (segment (start 97.995 43) (end 97.995 57.505) (width 0.5) (layer "B.Cu") (net 21))
   (segment (start 91.5 69.5) (end 91 70) (width 0.5) (layer "B.Cu") (net 21))
-  (via (at 90.5 93) (size 0.8) (drill 0.4) (layers "F.Cu" "B.Cu") (net 22))
   (segment (start 87.5 102.5) (end 85.5 102.5) (width 0.5) (layer "B.Cu") (net 22))
   (segment (start 87.5 101) (end 90.5 98) (width 0.5) (layer "B.Cu") (net 22))
@@
   (segment (start 104 49.5) (end 113 49.5) (width 1) (layer "F.Cu") (net 23))
   (segment (start 97.5 65) (end 99.5 63) (width 1) (layer "F.Cu") (net 23))
-  (segment (start 103.9 49.5) (end 103.9 49.6) (width 1) (layer "F.Cu") (net 23))
   (segment (start 95 65) (end 97.5 65) (width 1) (layer "F.Cu") (net 23))
   (segment (start 89.6 80.4) (end 88 80.4) (width 0.5) (layer "F.Cu") (net 24))
@@
   (segment (start 85 52) (end 83 54) (width 0.5) (layer "B.Cu") (net 31))
   (segment (start 103.5 52.5) (end 103 52) (width 0.5) (layer "B.Cu") (net 31))
-  (segment (start 92 104) (end 87.5 104) (width 0.5) (layer "F.Cu") (net 32))
+  (segment (start 91.85 104.15) (end 92 104) (width 0.5) (layer "B.Cu") (net 32))
+  (segment (start 87.5 104.15) (end 91.85 104.15) (width 0.5) (layer "B.Cu") (net 32))
   (segment (start 83.68 75.32) (end 88 75.32) (width 0.5) (layer "F.Cu") (net 36))
   (segment (start 81.5 86.85) (end 81.5 77.5) (width 0.5) (layer "F.Cu") (net 36))
@@
   (segment (start 84.14 77.86) (end 88 77.86) (width 0.5) (layer "F.Cu") (net 37))
   (segment (start 79 83.5) (end 79 83) (width 0.5) (layer "F.Cu") (net 37))
-  (segment (start 87.86 78) (end 88 77.86) (width 0.5) (layer "F.Cu") (net 37))
   (segment (start 79 87) (end 79 83.5) (width 0.5) (layer "F.Cu") (net 37))
   (segment (start 82.5 79.5) (end 84.14 77.86) (width 0.5) (layer "F.Cu") (net 37))
@@
   (segment (start 81.5 94.035) (end 81.5 88.5) (width 0.5) (layer "F.Cu") (net 40))
   (segment (start 81.59 94.125) (end 81.5 94.035) (width 0.5) (layer "F.Cu") (net 40))
-  (zone (net 0) (net_name "") (layer "F.Cu") (hatch none 0.5)
+  (zone (net 1) (net_name "GND") (layer "F.Cu") (hatch none 0.5)
     (connect_pads (clearance 0.5))
     (min_thickness 0.25) (filled_areas_thickness no)
